Commit message: Modify urdf and add moveit config.

File: sp_robot_description/robots/sp_robot.urdf (robot description, URDF)
Before this commit: robot sp_robot_description, 3 links, 2 joints
Links:
- added link link_eef, mass 4.90182522957532; collision mesh filename=package://sp_robot_description/meshes/link_eef.STL; visual mesh filename=package://sp_robot_description/meshes/link_eef.STL
- link base_link: mass 4.5128902913737 -> 4.51289029137366
- link link1: mass 5.8092 -> 5.80923663996572
- link link2: mass 5.8092 -> 5.80923663996572
Joints:
- added joint joint_eef: type continuous, parent link2, child link_eef, origin xyz=0.6 0 0.152 rpy=0 0 0, axis 0 0 -1
- joint joint1: origin xyz=0 0 0.092 rpy=0 0 0.39881 -> xyz=0 0 0.092 rpy=0 0 0
- joint joint2: origin xyz=0.6 0 0.052 rpy=0 0 -0.84687 -> xyz=0.6 0 0.052 rpy=0 0 0
